File: EAGLE/pwm-logger.sch (EAGLE design)
At the start: 29 parts, among them U1 24LC256, U2 3.3V/150mA

Commit message: Updated schematics
Parts:
- added C1: 330UF-POLAR, SparkFun-Capacitors:330UF-POLAR
- Y1: value (none) -> 5 MHz
- renumbered PROPELLER to U$1
Connections:
- net POWER_IN: now also U2.EN
- net VDD: now also C1.+
- net VSS: now also C1.-, U2.BP; no longer U2.EN
Other:
- note added: "0.0.1"
- note removed: "0"
